File: Flight Controller PCB/drone_sensors.kicad_sch (KiCad schematic)
At the start: 5 parts, among them U3 LSM6DSRXTR, U4 BMP585

Commit message: Finished converters, combined converter & sensor sheets. Updated I2C & CS pullups. TODO: Add motor control pins to MCU & control pins for camera
Parts:
- removed C18, C19, C20: 100nF, Capacitor_SMD:C_0603_1608Metric, symbol Device:C
- removed U3: LSM6DSRXTR, Drone_Fp:LGA-14L_STM, symbol Drone_sym:LSM6DSRXTR
- removed U4: BMP585, Drone_Fp:LGA9_BMP585_BOS, symbol Drone_sym:BMP585
Connections:
- no-connect marks 3 -> 0
Other:
- note removed: "ACCELEROMETER"
- note removed: "PRESSURE SENSOR"
