File: Flight Controller PCB/drone_bms.kicad_sch (KiCad schematic)
At the start: 13 parts, among them J1 BATT_JST, J3 USB_C_Receptacle, Q1 Si1442DH, U1 BQ29200DRBR

Commit message: Some changes. TODO: Add power and control for RunCam2. Add battery voltage monitoring
Changed lines of the file:
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@@
 	)
 	(hierarchical_label "VBATT"
-		(shape input)
+		(shape output)
 		(at 213.36 30.48 0)
 		(effects

Commit message: Init
Parts:
- added J4: BATT_XT30, Connector_AMASS:AMASS_XT30PW-M_1x02_P2.50mm_Horizontal, symbol Connector_Generic:Conn_01x02
- added R14, R15: 5k1, Resistor_SMD:R_0603_1608Metric, symbol Device:R_US
Connections:
- net GND: now also J3.A1 (GND), J3.A12 (GND), J3.B1 (GND), J3.B12 (GND), J3.SH (SHIELD), J4.1 (Pin_1), R14.1, R15.1
- net VBATT: now also J4.2 (Pin_2)
- net C2: now reaches J1.1 (Pin_1), R3.1
- net C1: now reaches J1.2 (Pin_2), R1.1, R2.1
- net +5V: now reaches J3.A4 (VBUS), J3.A9 (VBUS), J3.B4 (VBUS), J3.B9 (VBUS)
- net USB_CC1: now reaches J3.A5 (CC1)
- net USB_CC1: now also R14.2
- net USB_D+: now reaches J3.A6 (D+)
- net USB_D+: now also J3.B6 (D+)
- net USB_D-: now reaches J3.A7 (D-)
- net USB_D-: now also J3.B7 (D-)
- net USB_CC2: now reaches J3.B5 (CC2)
- net USB_CC2: now also R15.2
- no-connect marks 0 -> 10
Other:
- note added: "XT30 Battery Input"
- moved on the sheet: C1, C2, C3, C4, J1, Q1, R1, R2, R3, R4, R5, U1
